File: EGPad.sch (KiCad schematic (older format))
At the start: 59 parts, among them SW1 Rotary_Encoder_Switch, SW2 Rotary_Encoder_Switch, SW3 Rotary_Encoder_Switch, U1 ProMicro

Commit message: adding oled from Corne style and reverse PCB
Parts:
- removed U1: ProMicro, Keebio Footprints:ArduinoProMicro-Mini-USB, symbol keebio:ProMicro
- added J1: OLED, kbd:OLED, symbol Connector_Generic:Conn_01x04
- added JP1, JP2, JP3, JP4: Jmp, kbd:Jumper, symbol Device:Jumper_NO_Small
- added R13, R14: R, kbd:R, symbol Device:R_Small
- added RSW1: SW_Push, kbd:ResetSW, symbol Switch:SW_Push
- added U1: ProMicro, kbd:ProMicro_v2, symbol kbd:ProMicro
- MX1, MX10, MX11, MX12, MX13, MX14, MX15, MX16, MX17, MX2, MX3, MX4, MX5, MX6, MX7, MX8, MX9: symbol MX_Alps_Hybrid:MX-NoLED -> EGPad-rescue:MX-NoLED-MX_Alps_Hybrid
Connections:
- net labels added: SCL, SDA, reset
- wire segments 126 -> 152
- no-connect marks 6 -> 1

Commit message: optimization and gerber for production
Parts:
- added JP5, JP6, JP7, JP8: Jmp, kbd:Jumper, symbol Device:Jumper_NO_Small
Connections:
- net GND: now also JP8.2
- net SCL: now also JP6.2
- net SDA: now also JP5.2
- net VCC: now also JP7.2
- net at J1.1 (Pin_1), JP4.1: now also JP8.1
- net at J1.2 (Pin_2), JP3.1: now also JP7.1
- net at J1.3 (Pin_3), JP2.1: now also JP6.1
- net at J1.4 (Pin_4), JP1.1: now also JP5.1
Changed lines of the file:
@@
 	1850 3500 1850 3800
 Wire Wire Line
-	1350 3500 1850 3500
+	1350 3500 1400 3500
+$Comp
+L Device:Jumper_NO_Small JP5
+U 1 1 617D641B
+P 2050 4100
+F 0 "JP5" H 2050 4150 50  0000 C CNN
+F 1 "Jmp" H 2050 4050 50  0000 C CNN
+F 2 "kbd:Jumper" H 2050 4100 50  0001 C CNN
+F 3 "~" H 2050 4100 50  0001 C CNN
+	1    2050 4100
+	1    0    0    -1
+$EndComp
+$Comp
+L Device:Jumper_NO_Small JP6
+U 1 1 617D6A57
+P 2050 4300
+F 0 "JP6" H 2050 4350 50  0000 C CNN
+F 1 "Jmp" H 2050 4250 50  0000 C CNN
+F 2 "kbd:Jumper" H 2050 4300 50  0001 C CNN
+F 3 "~" H 2050 4300 50  0001 C CNN
+	1    2050 4300
+	1    0    0    -1
+$EndComp
+$Comp
+L Device:Jumper_NO_Small JP7
+U 1 1 617D708C
+P 2050 4500
+F 0 "JP7" H 2050 4550 50  0000 C CNN
+F 1 "Jmp" H 2050 4450 50  0000 C CNN
+F 2 "kbd:Jumper" H 2050 4500 50  0001 C CNN
+F 3 "~" H 2050 4500 50  0001 C CNN
+	1    2050 4500
+	1    0    0    -1
+$EndComp
+$Comp
+L Device:Jumper_NO_Small JP8
+U 1 1 617D74C5
+P 2050 4700
+F 0 "JP8" H 2050 4750 50  0000 C CNN
+F 1 "Jmp" H 2050 4650 50  0000 C CNN
+F 2 "kbd:Jumper" H 2050 4700 50  0001 C CNN
+F 3 "~" H 2050 4700 50  0001 C CNN
+	1    2050 4700
+	1    0    0    -1
+$EndComp
+Text GLabel 2250 4100 2    50   Input ~ 0
+SDA
+Text GLabel 2250 4300 2    50   Input ~ 0
+SCL
+$Comp
+L power:VCC #PWR0111
+U 1 1 617D7A52
+P 2250 4500
+F 0 "#PWR0111" H 2250 4350 50  0001 C CNN
+F 1 "VCC" V 2265 4628 50  0000 L CNN
+F 2 "" H 2250 4500 50  0001 C CNN
+F 3 "" H 2250 4500 50  0001 C CNN
+	1    2250 4500
+	0    1    1    0
+$EndComp
+$Comp
+L power:GND #PWR0112
+U 1 1 617D7E40
+P 2250 4700
+F 0 "#PWR0112" H 2250 4450 50  0001 C CNN
+F 1 "GND" V 2255 4572 50  0000 R CNN
+F 2 "" H 2250 4700 50  0001 C CNN
+F 3 "" H 2250 4700 50  0001 C CNN
+	1    2250 4700
+	0    -1   -1   0
+$EndComp
 Wire Wire Line
-	1350 3200 1950 3200
+	2150 4100 2250 4100
 Wire Wire Line
-	1350 3300 1950 3300
+	2150 4300 2250 4300
 Wire Wire Line
-	1350 3400 1900 3400
+	2150 4500 2250 4500
+Wire Wire Line
+	1350 3400 1500 3400
+Wire Wire Line
+	1350 3300 1600 3300
+Wire Wire Line
+	1350 3200 1700 3200
+Wire Wire Line
+	1700 3200 1700 4100
+Wire Wire Line
+	1700 4100 1950 4100
+Connection ~ 1700 3200
+Wire Wire Line
+	1700 3200 1950 3200
+Wire Wire Line
+	1600 3300 1600 4300
+Wire Wire Line
+	1600 4300 1950 4300
+Connection ~ 1600 3300
+Wire Wire Line
+	1600 3300 1950 3300
+Wire Wire Line
+	1500 3400 1500 4500
+Wire Wire Line
+	1500 4500 1950 4500
+Connection ~ 1500 3400
+Wire Wire Line
+	1500 3400 1900 3400
+Wire Wire Line
+	1400 3500 1400 4700
+Wire Wire Line
+	1400 4700 1950 4700
+Connection ~ 1400 3500
+Wire Wire Line
+	1400 3500 1850 3500
+Wire Wire Line
+	2150 4700 2250 4700
 $EndSCHEMATC
